File: Eagle/preamp/preamp.sch (EAGLE design)
At the start: 25 parts, among them J1 61300411121, J2 61300411121, J3 61300411121, J4 61300411121, J5 61300411121, U1 LM358

Commit message: eagle更新
Other:
- note added: "「preampでによる増幅の直後の信号」計測位置"
Changed lines of the file:
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@@
 <text x="5.08" y="88.9" size="1.778" layer="91">0.27u</text>
 <text x="10.16" y="-12.7" size="1.778" layer="91">0.27u</text>
+<text x="93.98" y="83.82" size="1.778" layer="91">「preampでによる増幅の直後の信号」計測位置</text>
 </plain>
 <instances>
