File: Eagle/filter+preamp/150HzLPF_8GainPreamp.brd (EAGLE design)
At the start: 76.2 x 37.8 mm, 19 parts, among them U1 LM358, U2 LM358

Commit message: final ver.
Parts:
- C8, C9: value ??? -> 33u
- moved C9 3.83 mm to (46.4, 19.7), flipped to the bottom
- moved C8 3.61 mm to (21.8, 18.6), flipped to the bottom
Routing:
- net N$6: track 55.2 -> 148.5 mm
- net N$7: track 75.1 -> 32.1 mm
- net N$17: track 168.0 -> 172.0 mm
- net N$4: track 18.5 -> 17.5 mm
- net N$3: track 11.5 -> 12.0 mm
