File: Eagle/filter+preamp/150HzLPF_8GainPreamp.brd (EAGLE design)
At the start: 76.2 x 37.8 mm, 19 parts, among them U1 LM358, U2 LM358

Commit message: add LED
Routing:
- net N$17: track 172.0 -> 0.00 mm
- net N$6: track 148.5 -> 0.00 mm
- net N$15: track 76.0 -> 0.00 mm
- net N$7: track 32.1 -> 0.00 mm
- net N$10: track 30.8 -> 0.00 mm
- net N$5: track 26.1 -> 0.00 mm
- net N$4: track 17.5 -> 0.00 mm
- net N$2: track 17.5 -> 0.00 mm
- net N$8: track 16.6 -> 0.00 mm
- net N$9: track 16.3 -> 0.00 mm
- net N$11: track 12.2 -> 0.00 mm
- net N$3: track 12.0 -> 0.00 mm
- net N$13: track 10.3 -> 0.00 mm
- net N$1: track 7.76 -> 0.00 mm

Commit message: consistent error
Parts:
- removed 10V-18V_SUPPLY_FOR_OPEAMP: 1X4-3.5MM, adafruit:1X04-3.5MM
- added 18V_SHARE, 18V_SUPPLY_FOR_OPEAMP: (no value), pinhead:1X03
- added 5V_SHARE: (no value), pinhead:1X02
- added D2, D3: LTL-1CHE, LED:RADIAL_3MM
- added R8, R9: 700k, rcl:0207/7
- 5V_SUPPLY_FOR_SENSOR, SENSOR_OUTPUT: value 1X4-3.5MM -> (none); device adafruit:1X04-3.5MM -> pinhead:1X02
- SENSOR_INPUT: value 1X4-3.5MM -> (none); device adafruit:1X04-3.5MM -> pinhead:1X04
- moved 5V_SUPPLY_FOR_SENSOR 109.7 mm to (-35.6, 39.4), turned to 0 degrees
- moved R2 98.2 mm to (-33.0, 50.8)
- moved C5 91.8 mm to (-45.7, 6.35)
- moved R6 89.8 mm to (-27.9, 55.9), turned to 0 degrees
- moved C1 88.4 mm to (-26.7, 25.4), turned to 0 degrees
- moved C2 86.9 mm to (-35.6, 25.4), turned to 0 degrees
- moved R4 83.6 mm to (-53.3, 50.8), turned to 0 degrees
- moved C8 82.3 mm to (-55.9, 45.7), flipped to the top, turned to 0 degrees
- moved R5 81.6 mm to (-17.8, 55.9), turned to 0 degrees
- moved R3 72.2 mm to (-43.2, 50.8), turned to 0 degrees
- moved C9 70.8 mm to (-16.5, 52.1), flipped to the top, turned to 0 degrees
- moved C4 68.6 mm to (-33.0, 6.35), turned to 0 degrees
- moved R1 68.5 mm to (-22.9, 50.8)
- moved C3 41.6 mm to (-20.3, 6.35), turned to 0 degrees
- moved SENSOR_OUTPUT 21.9 mm to (5.08, 6.35)
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Connections:
- new net N$12: D2.A, R8.1
- new net N$16: D3.A, R9.2
- net N$15: now also 5V_SHARE.2, R8.2; no longer 5V_SUPPLY_FOR_SENSOR.4
- net N$17: now also 18V_SHARE.2, 18V_SUPPLY_FOR_OPEAMP.2, 5V_SHARE.1, D2.C, D3.C; no longer 10V-18V_SUPPLY_FOR_OPEAMP.1, 10V-18V_SUPPLY_FOR_OPEAMP.3, 5V_SUPPLY_FOR_SENSOR.3
- net N$6: now also 18V_SHARE.3, 18V_SUPPLY_FOR_OPEAMP.3, R9.1; no longer 10V-18V_SUPPLY_FOR_OPEAMP.2, 10V-18V_SUPPLY_FOR_OPEAMP.4
Routing:
- removed copper zone on layer 16, net GND
Other:
- board size 76.2 x 37.8 mm -> 160 x 100 mm
